Commit message: updated units to mm for stl models and all urdf primitives and refs. Inertias are not in kg*m^2, masses in kg. Displays nicely on online viewers

File: MATLAB/ability_hand.urdf (robot description, URDF)
Before this commit: robot ability_hand, 11 links, 10 joints
Links:
- link base: geometry visual cylinder length=25.000001e-3 radius=3.500000e-3; visual cylinder length=25.000660e-3 radius=3.500000e-3
- link index_L1: geometry visual box size=38.6070382e-3 4e-3 4e-3; visual mesh filename=models/idx-F1.STL
- link index_L2: geometry visual box size=35.41e-3 4e-3 4e-3; visual cylinder length=3e-3 radius=4e-3
- link middle_L1: geometry visual box size=38.6070382e-3 4e-3 4e-3; visual mesh filename=models/idx-F1.STL
- link middle_L2: geometry visual box size=35.41e-3 4e-3 4e-3; visual cylinder length=3e-3 radius=4e-3
- link pinky_L1: geometry visual box size=38.6070382e-3 4e-3 4e-3; visual mesh filename=models/idx-F1.STL
- link pinky_L2: geometry visual box size=35.41e-3 4e-3 4e-3; visual cylinder length=3e-3 radius=4e-3
- link ring_L1: geometry visual box size=38.6070382e-3 4e-3 4e-3; visual mesh filename=models/idx-F1.STL
- link ring_L2: geometry visual box size=35.41e-3 4e-3 4e-3; visual cylinder length=3e-3 radius=4e-3
- link thumb_L1: geometry visual box size=31.15246724e-3 5e-3 4e-3; visual mesh filename=models/thumb-F1.STL
- link thumb_L2: geometry visual box size=60.93e-3 4e-3 8e-3; visual cylinder length=7e-3 radius=7e-3
Joints:
- joint index_q1: origin xyz=-9.49 -13.04 -62.95 rpy=-1.982050 1.284473 -2.090591 -> xyz=-9.49e-3 -13.04e-3 -62.95e-3 rpy=-1.982050 1.284473 -2.090591
- joint index_q2: origin xyz=38.472723 3.257695 0.000000 rpy=0 0 0.084474 -> xyz=38.472723e-3 3.257695e-3 0.000000e-3 rpy=0 0 0.084474
- joint middle_q1: origin xyz=9.653191 -15.310271 -67.853949 rpy=-1.860531 1.308458 -1.896217 -> xyz=9.653191e-3 -15.310271e-3 -67.853949e-3 rpy=-1.860531 1.308458 -1.896217
- joint middle_q2: origin xyz=38.472723 3.257695 0.000000 rpy=0 0 0.084474 -> xyz=38.472723e-3 3.257695e-3 0.000000 rpy=0 0 0.084474
- joint pinky_q1: origin xyz=49.521293 -11.004583 -63.029065 rpy=-1.765110 1.322220 -1.658383 -> xyz=49.521293e-3 -11.004583e-3 -63.029065e-3 rpy=-1.765110 1.322220 -1.658383
- joint pinky_q2: origin xyz=38.472723 3.257695 0.000000 rpy=0 0 0.084474 -> xyz=38.472723e-3 3.257695e-3 0.000000 rpy=0 0 0.084474
- joint ring_q1: origin xyz=29.954260 -14.212492 -67.286105 rpy=-1.716598 1.321452 -1.675862 -> xyz=29.954260e-3 -14.212492e-3 -67.286105e-3 rpy=-1.716598 1.321452 -1.675862
- joint ring_q2: origin xyz=38.472723 3.257695 0.000000 rpy=0 0 0.084474 -> xyz=38.472723e-3 3.257695e-3 0.000000 rpy=0 0 0.084474
- joint thumb_q2: origin xyz=27.8283501 0 -14.7507000 rpy=4.450589592585541 0 0 -> xyz=27.8283501e-3 0 -14.7507000e-3 rpy=4.450589592585541 0 0

Commit message: fixed abh 4bar and changed the display limits

File: MATLAB/ability_hand.urdf (robot description, URDF)
Before this commit: robot ability_hand, 11 links, 10 joints
Joints:
- joint index_q1: limit (none) -> lower=0 upper=2.0943951 effort=0.20 velocity=8.0677777442; type continuous -> revolute
- joint index_q2: limit (none) -> lower=0.0 upper=2.6586 effort=0.20 velocity=8.0677777442; type continuous -> revolute
- joint middle_q1: limit (none) -> lower=0 upper=2.0943951 effort=0.20 velocity=8.0677777442; type continuous -> revolute
- joint middle_q2: limit (none) -> lower=0.0 upper=2.6586 effort=0.20 velocity=8.0677777442; type continuous -> revolute
- joint pinky_q1: limit (none) -> lower=0 upper=2.0943951 effort=0.20 velocity=8.0677777442; type continuous -> revolute
- joint pinky_q2: limit (none) -> lower=0.0 upper=2.6586 effort=0.20 velocity=8.0677777442; type continuous -> revolute
- joint ring_q1: limit (none) -> lower=0 upper=2.0943951 effort=0.20 velocity=8.0677777442; type continuous -> revolute
- joint ring_q2: limit (none) -> lower=0.0 upper=2.6586 effort=0.20 velocity=8.0677777442; type continuous -> revolute
- joint thumb_q1: limit (none) -> lower=-2.0943951 upper=0 effort=0.20 velocity=8.0677777442; type continuous -> revolute
- joint thumb_q2: limit (none) -> lower=0 upper=2.0943951 effort=0.20 velocity=8.0677777442; type continuous -> revolute
