Commit message: added new wrist piece

File: URDF/ability_hand.urdf (robot description, URDF)
Before this commit: robot ability_hand, 11 links, 10 joints
Links:
- link base: geometry visual cylinder length=25.000001e-3 radius=3.500000e-3; visual cylinder length=25.000660e-3 radius=3.500000e-3

Commit message: removed geometric primitives and added name properties to hand meshes

File: URDF/ability_hand.urdf (robot description, URDF)
Before this commit: robot ability_hand, 11 links, 10 joints
Links:
- link base: geometry visual mesh filename=models/FB_palm_ref.STL; visual mesh filename=models/WRISTADAPTER.STL
- link index_L1: geometry visual mesh filename=models/idx-F1.STL
- link index_L2: geometry visual mesh filename=models/idx-F2.STL
- link middle_L1: geometry visual mesh filename=models/idx-F1.STL
- link middle_L2: geometry visual mesh filename=models/idx-F2.STL
- link pinky_L1: geometry visual mesh filename=models/idx-F1.STL
- link pinky_L2: geometry visual mesh filename=models/idx-F2.STL
- link ring_L1: geometry visual mesh filename=models/idx-F1.STL
- link ring_L2: geometry visual mesh filename=models/idx-F2.STL
- link thumb_L1: geometry visual mesh filename=models/thumb-F1.STL
- link thumb_L2: geometry visual mesh filename=models/thumb-F2.STL
