Commit message: added wrist update to right hand also

File: URDF/ability_hand_right.urdf (robot description, URDF)
Before this commit: robot ability_hand, 11 links, 10 joints
Links:
- link base: geometry visual mesh filename=models/FB_palm_ref_MIR.STL; visual mesh filename=models/wristmesh.STL

Commit message: base frame update, using wrist frame

File: URDF/ability_hand_right.urdf (robot description, URDF)
Before this commit: robot ability_hand, 11 links, 10 joints
Links:
- added link wrist; visual mesh filename=models/wristmesh.STL
- link base: geometry visual mesh filename=models/FB_palm_ref_MIR.STL
Joints:
- added joint wrist2thumb: type fixed, parent wrist, child base, origin xyz=-24.0476665e-3 3.78124745e-3 32.32964923e-3 rpy=3.14148426 -0.08848813 -3.14036612

Commit message: added bogus inertial info to the wrist

File: URDF/ability_hand_right.urdf (robot description, URDF)
Before this commit: robot ability_hand, 12 links, 11 joints
Links:
- link base: mass 0.400 -> 0.200
- link wrist: mass None -> 0.200

Commit message: len with e-3 append

File: URDF/ability_hand_right.urdf (robot description, URDF)
Before this commit: robot ability_hand, 17 links, 16 joints
Joints:
- joint index_q1: origin xyz= 0.00949 -0.01304 -0.06295  rpy= -1.1595426535897932 1.284473 -1.0510016535897932  -> xyz= 9.49e-3 -13.04e-3 -62.95e-3  rpy= -1.1595426535897932 1.284473 -1.0510016535897932 
- joint middle_q1: origin xyz= -0.009653191 -0.015310271 -0.067853949  rpy= -1.2810616535897934 1.308458 -1.2453756535897933  -> xyz= -9.653191e-3 -15.310271e-3 -67.853949e-3  rpy= -1.2810616535897934 1.308458 -1.2453756535897933 
- joint pinky_q1: origin xyz= -0.049521293 -0.011004583 -0.063029065  rpy= -1.3764826535897934 1.32222 -1.4832096535897932  -> xyz= -49.521293e-3 -11.004583e-3 -63.029065e-3  rpy= -1.3764826535897934 1.32222 -1.4832096535897932 
- joint ring_q1: origin xyz= -0.02995426 -0.014212492 -0.067286105  rpy= -1.424994653589793 1.321452 -1.4657306535897934  -> xyz= -29.95426e-3 -14.212492e-3 -67.286105e-3  rpy= -1.424994653589793 1.321452 -1.4657306535897934 
- joint thumb_q2: origin xyz= 0.0278283501 1.7436510745838653e-19 0.0147507  rpy= 1.832595714594045 -0.0 5.366520605522463e-18  -> xyz= 27.8283501e-3 1.7436510745838653e-19 14.7507e-3  rpy= 1.832595714594045 -0.0 5.366520605522463e-18 
