Commit message: added mimic based on best-fit line to the curve of the true 4bar linkage relationship

File: URDF/ability_hand_left.urdf (robot description, URDF)
Before this commit: robot ability_hand, 11 links, 10 joints
Joints:
- joint index_q2: mimic (none) -> joint=index_q1 multiplier=1.061707401078210 offset=0.565475650708972
- joint middle_q2: mimic (none) -> joint=middle_q1 multiplier=1.061707401078210 offset=0.565475650708972
- joint pinky_q2: mimic (none) -> joint=pinky_q1 multiplier=1.061707401078210 offset=0.565475650708972
- joint ring_q2: mimic (none) -> joint=ring_q1 multiplier=1.061707401078210 offset=0.565475650708972

File: URDF/ability_hand_right.urdf (robot description, URDF)
Before this commit: robot ability_hand, 11 links, 10 joints
Joints:
- joint index_q2: mimic (none) -> joint=index_q1 multiplier=1.061707401078210 offset=0.565475650708972
- joint middle_q2: mimic (none) -> joint=middle_q1 multiplier=1.061707401078210 offset=0.565475650708972
- joint pinky_q2: mimic (none) -> joint=pinky_q1 multiplier=1.061707401078210 offset=0.565475650708972
- joint ring_q2: mimic (none) -> joint=ring_q1 multiplier=1.061707401078210 offset=0.565475650708972

Commit message: updated urdf files with improved mimic linear estimation based on the updated frame reference math integrated into the 4bar linkages calculations. the calculation of these parameters is provided in a separate python file, which also shows error behavior

File: URDF/ability_hand_left.urdf (robot description, URDF)
Before this commit: robot ability_hand, 11 links, 10 joints
Joints:
- joint index_q2: mimic joint=index_q1 multiplier=1.061707401078210 offset=0.565475650708972 -> joint=index_q1 multiplier=1.05851325 offset=0.72349796
- joint middle_q2: mimic joint=middle_q1 multiplier=1.061707401078210 offset=0.565475650708972 -> joint=middle_q1 multiplier=1.05851325 offset=0.72349796
- joint pinky_q2: mimic joint=pinky_q1 multiplier=1.061707401078210 offset=0.565475650708972 -> joint=pinky_q1 multiplier=1.05851325 offset=0.72349796
- joint ring_q2: mimic joint=ring_q1 multiplier=1.061707401078210 offset=0.565475650708972 -> joint=ring_q1 multiplier=1.05851325 offset=0.72349796

File: URDF/ability_hand_right.urdf (robot description, URDF)
Before this commit: robot ability_hand, 11 links, 10 joints
Joints:
- joint index_q2: mimic joint=index_q1 multiplier=1.061707401078210 offset=0.565475650708972 -> joint=index_q1 multiplier=1.05851325 offset=0.72349796
- joint middle_q2: mimic joint=middle_q1 multiplier=1.061707401078210 offset=0.565475650708972 -> joint=middle_q1 multiplier=1.05851325 offset=0.72349796
- joint pinky_q2: mimic joint=pinky_q1 multiplier=1.061707401078210 offset=0.565475650708972 -> joint=pinky_q1 multiplier=1.05851325 offset=0.72349796
- joint ring_q2: mimic joint=ring_q1 multiplier=1.061707401078210 offset=0.565475650708972 -> joint=ring_q1 multiplier=1.05851325 offset=0.72349796

Commit message: used updated wristmesh and frame definition in left hand.

File: URDF/ability_hand_left.urdf (robot description, URDF)
Before this commit: robot ability_hand, 11 links, 10 joints
Links:
- link base: geometry visual mesh filename=models/FB_palm_ref.STL; visual mesh filename=models/wristmesh.STL

Commit message: left hand base frame is wrist

File: URDF/ability_hand_left.urdf (robot description, URDF)
Before this commit: robot ability_hand, 11 links, 10 joints
Links:
- added link wrist, mass 0.200; visual mesh filename=models/wristmesh.STL
Joints:
- added joint wrist2thumb: type fixed, parent wrist, child base, origin xyz=24.0476665e-3 3.78124745e-3 32.32964923e-3 rpy=3.14148426 0.08848813 3.14036612

Commit message: link names, etc

File: URDF/ability_hand_left.urdf (robot description, URDF)
Before this commit: robot ability_hand, 12 links, 11 joints
Links:
- removed link wrist
- added link thumb_base, mass 0.400; visual mesh filename=models/FB_palm_ref.STL; visual mesh filename=models/wristmesh.STL
- link base: mass 0.400 -> 0.200; geometry visual mesh filename=models/wristmesh.STL
Joints:
- joint index_q1: parent base -> thumb_base
- joint middle_q1: parent base -> thumb_base
- joint pinky_q1: parent base -> thumb_base
- joint ring_q1: parent base -> thumb_base
- joint thumb_q1: parent base -> thumb_base
- joint wrist2thumb: child base -> thumb_base; parent wrist -> base

File: URDF/ability_hand_right.urdf (robot description, URDF)
Before this commit: robot ability_hand, 12 links, 11 joints
Links:
- removed link wrist
- added link thumb_base, mass 0.200; visual mesh filename=models/FB_palm_ref_MIR.STL
- link base: geometry visual mesh filename=models/wristmesh.STL
Joints:
- joint index_q1: parent base -> thumb_base
- joint middle_q1: parent base -> thumb_base
- joint pinky_q1: parent base -> thumb_base
- joint ring_q1: parent base -> thumb_base
- joint thumb_q1: parent base -> thumb_base
- joint wrist2thumb: child base -> thumb_base; parent wrist -> base

Commit message: added anchor points to fingertips

File: URDF/ability_hand_left.urdf (robot description, URDF)
Before this commit: robot ability_hand, 12 links, 11 joints
Links:
- added link index_anchor
- added link middle_anchor
- added link pinky_anchor
- added link ring_anchor
Joints:
- added joint idx_anchor: type fixed, parent index_L2, child index_anchor, origin xyz=0.02243 -0.01044 0.00014 rpy=0 0 0
- added joint mid_anchor: type fixed, parent middle_L2, child middle_anchor, origin xyz=0.02243 -0.01044 0.00014 rpy=0 0 0
- added joint pnky_anchor: type fixed, parent pinky_L2, child pinky_anchor, origin xyz=0.02243 -0.01044 0.00014 rpy=0 0 0
- added joint rng_anchor: type fixed, parent ring_L2, child ring_anchor, origin xyz=0.02243 -0.01044 0.00014 rpy=0 0 0

File: URDF/ability_hand_right.urdf (robot description, URDF)
Before this commit: robot ability_hand, 12 links, 11 joints
Links:
- added link index_anchor
- added link middle_anchor
- added link pinky_anchor
- added link ring_anchor
Joints:
- added joint idx_anchor: type fixed, parent index_L2, child index_anchor, origin xyz=0.02243 -0.01044 0.00014 rpy=0 0 0
- added joint mid_anchor: type fixed, parent middle_L2, child middle_anchor, origin xyz=0.02243 -0.01044 0.00014 rpy=0 0 0
- added joint pnky_anchor: type fixed, parent pinky_L2, child pinky_anchor, origin xyz=0.02243 -0.01044 0.00014 rpy=0 0 0
- added joint rng_anchor: type fixed, parent ring_L2, child ring_anchor, origin xyz=0.02243 -0.01044 0.00014 rpy=0 0 0

Commit message: centimeters urdf

File: URDF/ability_hand_left.urdf (robot description, URDF)
Before this commit: robot ability_hand, 12 links, 11 joints
Links:
- link base: geometry visual mesh filename=models/wristmesh.STL scale=10 10 10
- link index_L1: geometry visual mesh filename=models/idx-F1.STL scale=10 10 10
- link index_L2: geometry visual mesh filename=models/idx-F2.STL scale=10 10 10
- link middle_L1: geometry visual mesh filename=models/idx-F1.STL scale=10 10 10
- link middle_L2: geometry visual mesh filename=models/idx-F2.STL scale=10 10 10
- link pinky_L1: geometry visual mesh filename=models/idx-F1.STL scale=10 10 10
- link pinky_L2: geometry visual mesh filename=models/idx-F2.STL scale=10 10 10
- link ring_L1: geometry visual mesh filename=models/idx-F1.STL scale=10 10 10
- link ring_L2: geometry visual mesh filename=models/idx-F2.STL scale=10 10 10
- link thumb_L1: geometry visual mesh filename=models/thumb-F1.STL scale=10 10 10
- link thumb_L2: geometry visual mesh filename=models/thumb-F2.STL scale=10 10 10
- link thumb_base: geometry visual mesh filename=models/FB_palm_ref.STL scale=10 10 10; visual mesh filename=models/wristmesh.STL scale=10 10 10
Joints:
- joint index_q1: origin xyz=-9.49e-3 -13.04e-3 -62.95e-3 rpy=-1.982050 1.284473 -2.090591 -> xyz=-9.49e-2 -13.04e-2 -62.95e-2 rpy=-1.982050 1.284473 -2.090591
- joint index_q2: origin xyz=38.472723e-3 3.257695e-3 0.000000e-3 rpy=0 0 0.084474 -> xyz=38.472723e-2 3.257695e-2 0.000000e-2 rpy=0 0 0.084474
- joint middle_q1: origin xyz=9.653191e-3 -15.310271e-3 -67.853949e-3 rpy=-1.860531 1.308458 -1.896217 -> xyz=9.653191e-2 -15.310271e-2 -67.853949e-2 rpy=-1.860531 1.308458 -1.896217
- joint middle_q2: origin xyz=38.472723e-3 3.257695e-3 0.000000 rpy=0 0 0.084474 -> xyz=38.472723e-2 3.257695e-2 0.000000 rpy=0 0 0.084474
- joint pinky_q1: origin xyz=49.521293e-3 -11.004583e-3 -63.029065e-3 rpy=-1.765110 1.322220 -1.658383 -> xyz=49.521293e-2 -11.004583e-2 -63.029065e-2 rpy=-1.765110 1.322220 -1.658383
- joint pinky_q2: origin xyz=38.472723e-3 3.257695e-3 0.000000 rpy=0 0 0.084474 -> xyz=38.472723e-2 3.257695e-2 0.000000 rpy=0 0 0.084474
- joint ring_q1: origin xyz=29.954260e-3 -14.212492e-3 -67.286105e-3 rpy=-1.716598 1.321452 -1.675862 -> xyz=29.954260e-2 -14.212492e-2 -67.286105e-2 rpy=-1.716598 1.321452 -1.675862
- joint ring_q2: origin xyz=38.472723e-3 3.257695e-3 0.000000 rpy=0 0 0.084474 -> xyz=38.472723e-2 3.257695e-2 0.000000 rpy=0 0 0.084474
- joint thumb_q2: origin xyz=27.8283501e-3 0 -14.7507000e-3 rpy=4.450589592585541 0 0 -> xyz=27.8283501e-2 0 -14.7507000e-2 rpy=4.450589592585541 0 0
- joint wrist2thumb: origin xyz=24.0476665e-3 3.78124745e-3 32.32964923e-3 rpy=3.14148426 0.08848813 3.14036612 -> xyz=24.0476665e-2 3.78124745e-2 32.32964923e-2 rpy=3.14148426 0.08848813 3.14036612

Commit message: cm to mm

File: URDF/ability_hand_left.urdf (robot description, URDF)
Before this commit: robot ability_hand, 16 links, 15 joints
Links:
- added link thumb_anchor
- link base: geometry visual mesh filename=models/wristmesh.STL
- link index_L1: geometry visual mesh filename=models/idx-F1.STL
- link index_L2: geometry visual mesh filename=models/idx-F2.STL
- link middle_L1: geometry visual mesh filename=models/idx-F1.STL
- link middle_L2: geometry visual mesh filename=models/idx-F2.STL
- link pinky_L1: geometry visual mesh filename=models/idx-F1.STL
- link pinky_L2: geometry visual mesh filename=models/idx-F2.STL
- link ring_L1: geometry visual mesh filename=models/idx-F1.STL
- link ring_L2: geometry visual mesh filename=models/idx-F2.STL
- link thumb_L1: geometry visual mesh filename=models/thumb-F1.STL
- link thumb_L2: geometry visual mesh filename=models/thumb-F2.STL
- link thumb_base: geometry visual mesh filename=models/FB_palm_ref.STL; visual mesh filename=models/wristmesh.STL
Joints:
- added joint thmb_anchor: type fixed, parent thumb_L2, child thumb_anchor, origin xyz=63.868144e-3  23.807059e-3 -3.629831e-3 rpy=0 0 0
- joint idx_anchor: origin xyz=0.02243 -0.01044 0.00014 rpy=0 0 0 -> xyz=31.5541e-3  -10.44e-3 0.14e-3 rpy=0 0 0
- joint index_q1: origin xyz=-9.49e-2 -13.04e-2 -62.95e-2 rpy=-1.982050 1.284473 -2.090591 -> xyz=-9.49e-3 -13.04e-3 -62.95e-3 rpy=-1.982050 1.284473 -2.090591
- joint index_q2: origin xyz=38.472723e-2 3.257695e-2 0.000000e-2 rpy=0 0 0.084474 -> xyz=38.472723e-3 3.257695e-3 0.000000e-3 rpy=0 0 0.084474
- joint mid_anchor: origin xyz=0.02243 -0.01044 0.00014 rpy=0 0 0 -> xyz=31.5541e-3  -10.44e-3 0.14e-3 rpy=0 0 0
- joint middle_q1: origin xyz=9.653191e-2 -15.310271e-2 -67.853949e-2 rpy=-1.860531 1.308458 -1.896217 -> xyz=9.653191e-3 -15.310271e-3 -67.853949e-3 rpy=-1.860531 1.308458 -1.896217
- joint middle_q2: origin xyz=38.472723e-2 3.257695e-2 0.000000 rpy=0 0 0.084474 -> xyz=38.472723e-3 3.257695e-3 0.000000 rpy=0 0 0.084474
- joint pinky_q1: origin xyz=49.521293e-2 -11.004583e-2 -63.029065e-2 rpy=-1.765110 1.322220 -1.658383 -> xyz=49.521293e-3 -11.004583e-3 -63.029065e-3 rpy=-1.765110 1.322220 -1.658383
- joint pinky_q2: origin xyz=38.472723e-2 3.257695e-2 0.000000 rpy=0 0 0.084474 -> xyz=38.472723e-3 3.257695e-3 0.000000 rpy=0 0 0.084474
- joint pnky_anchor: origin xyz=0.02243 -0.01044 0.00014 rpy=0 0 0 -> xyz=31.5541e-3  -10.44e-3 0.14e-3 rpy=0 0 0
- joint ring_q1: origin xyz=29.954260e-2 -14.212492e-2 -67.286105e-2 rpy=-1.716598 1.321452 -1.675862 -> xyz=29.954260e-3 -14.212492e-3 -67.286105e-3 rpy=-1.716598 1.321452 -1.675862
- joint ring_q2: origin xyz=38.472723e-2 3.257695e-2 0.000000 rpy=0 0 0.084474 -> xyz=38.472723e-3 3.257695e-3 0.000000 rpy=0 0 0.084474
- joint rng_anchor: origin xyz=0.02243 -0.01044 0.00014 rpy=0 0 0 -> xyz=31.5541e-3  -10.44e-3 0.14e-3 rpy=0 0 0
- joint thumb_q2: origin xyz=27.8283501e-2 0 -14.7507000e-2 rpy=4.450589592585541 0 0 -> xyz=27.8283501e-3 0 -14.7507000e-3 rpy=4.450589592585541 0 0
- joint wrist2thumb: origin xyz=24.0476665e-2 3.78124745e-2 32.32964923e-2 rpy=3.14148426 0.08848813 3.14036612 -> xyz=24.0476665e-3 3.78124745e-3 32.32964923e-3 rpy=3.14148426 0.08848813 3.14036612

Commit message: anchors for right hand

File: URDF/ability_hand_left.urdf (robot description, URDF)
Before this commit: robot ability_hand, 17 links, 16 joints
Links:
- link thumb_base: geometry visual mesh filename=models/FB_palm_ref.STL

File: URDF/ability_hand_right.urdf (robot description, URDF)
Before this commit: robot ability_hand, 16 links, 15 joints
Links:
- added link thumb_anchor
Joints:
- added joint thmb_anchor: type fixed, parent thumb_L2, child thumb_anchor, origin xyz=63.868144e-3  23.807059e-3 -3.629831e-3 rpy=0 0 0
- joint idx_anchor: origin xyz=0.02243 -0.01044 0.00014 rpy=0 0 0 -> xyz=31.5541e-3  -10.44e-3 0.14e-3 rpy=0 0 0
- joint mid_anchor: origin xyz=0.02243 -0.01044 0.00014 rpy=0 0 0 -> xyz=31.5541e-3  -10.44e-3 0.14e-3 rpy=0 0 0
- joint pnky_anchor: origin xyz=0.02243 -0.01044 0.00014 rpy=0 0 0 -> xyz=31.5541e-3  -10.44e-3 0.14e-3 rpy=0 0 0
- joint rng_anchor: origin xyz=0.02243 -0.01044 0.00014 rpy=0 0 0 -> xyz=31.5541e-3  -10.44e-3 0.14e-3 rpy=0 0 0

Commit message: fixed thumb anchor, again

File: URDF/ability_hand_left.urdf (robot description, URDF)
Before this commit: robot ability_hand, 17 links, 16 joints
Joints:
- joint thmb_anchor: origin xyz=63.868144e-3  23.807059e-3 -3.629831e-3 rpy=0 0 0 -> xyz=52.0012259e-3  28.0086971e-3 -.884835778e-3 rpy=0 0 0

File: URDF/ability_hand_right.urdf (robot description, URDF)
Before this commit: robot ability_hand, 17 links, 16 joints
Joints:
- joint thmb_anchor: origin xyz=63.868144e-3  23.807059e-3 -3.629831e-3 rpy=0 0 0 -> xyz=52.00122724e-3 28.00869333e-3 6.98483578e-3 rpy=0 0 0

Commit message: quick fixes for urdf and mujoco xml

File: URDF/ability_hand_left.urdf (robot description, URDF)
Before this commit: robot ability_hand, 17 links, 16 joints
Joints:
- joint index_q1: limit lower=0 upper=2.0943951 effort=0.20 velocity=8.0677777442 -> lower=0 upper=2.0943951 effort=6.0 velocity=8.0677777442
- joint index_q2: limit lower=0.0 upper=2.6586 effort=0.20 velocity=8.0677777442 -> lower=0.0 upper=2.6586 effort=6.0 velocity=8.0677777442
- joint middle_q1: limit lower=0 upper=2.0943951 effort=0.20 velocity=8.0677777442 -> lower=0 upper=2.0943951 effort=6.0 velocity=8.0677777442
- joint middle_q2: limit lower=0.0 upper=2.6586 effort=0.20 velocity=8.0677777442 -> lower=0.0 upper=2.6586 effort=6.0 velocity=8.0677777442
- joint pinky_q1: limit lower=0 upper=2.0943951 effort=0.20 velocity=8.0677777442 -> lower=0 upper=2.0943951 effort=6.0 velocity=8.0677777442
- joint pinky_q2: limit lower=0.0 upper=2.6586 effort=0.20 velocity=8.0677777442 -> lower=0.0 upper=2.6586 effort=6.0 velocity=8.0677777442
- joint ring_q1: limit lower=0 upper=2.0943951 effort=0.20 velocity=8.0677777442 -> lower=0 upper=2.0943951 effort=6.0 velocity=8.0677777442
- joint ring_q2: limit lower=0.0 upper=2.6586 effort=0.20 velocity=8.0677777442 -> lower=0.0 upper=2.6586 effort=6.0 velocity=8.0677777442
- joint thumb_q1: limit lower=-2.0943951 upper=0 effort=0.20 velocity=8.0677777442 -> lower=-2.0943951 upper=0 effort=1.2 velocity=40.338888721
- joint thumb_q2: limit lower=0 upper=2.0943951 effort=0.20 velocity=8.0677777442 -> lower=0 upper=2.0943951 effort=6.0 velocity=8.0677777442

File: URDF/ability_hand_right.urdf (robot description, URDF)
Before this commit: robot ability_hand, 17 links, 16 joints
Joints:
- joint index_q1: limit lower=0 upper=2.0943951 effort=0.20 velocity=8.0677777442 -> lower=0 upper=2.0943951 effort=6.0 velocity=8.0677777442
- joint index_q2: limit lower=0.0 upper=2.6586 effort=0.20 velocity=8.0677777442 -> lower=0.0 upper=2.6586 effort=6.0 velocity=8.0677777442
- joint middle_q1: limit lower=0 upper=2.0943951 effort=0.20 velocity=8.0677777442 -> lower=0 upper=2.0943951 effort=6.0 velocity=8.0677777442
- joint middle_q2: limit lower=0.0 upper=2.6586 effort=0.20 velocity=8.0677777442 -> lower=0.0 upper=2.6586 effort=6.0 velocity=8.0677777442
- joint pinky_q1: limit lower=0 upper=2.0943951 effort=0.20 velocity=8.0677777442 -> lower=0 upper=2.0943951 effort=6.0 velocity=8.0677777442
- joint pinky_q2: limit lower=0.0 upper=2.6586 effort=0.20 velocity=8.0677777442 -> lower=0.0 upper=2.6586 effort=6.0 velocity=8.0677777442
- joint ring_q1: limit lower=0 upper=2.0943951 effort=0.20 velocity=8.0677777442 -> lower=0 upper=2.0943951 effort=6.0 velocity=8.0677777442
- joint ring_q2: limit lower=0.0 upper=2.6586 effort=0.20 velocity=8.0677777442 -> lower=0.0 upper=2.6586 effort=6.0 velocity=8.0677777442
- joint thumb_q1: limit lower=-2.0943951 upper=0 effort=0.20 velocity=8.0677777442 -> lower=-2.0943951 upper=0 effort=1.2 velocity=40.338888721
- joint thumb_q2: limit lower=0 upper=2.0943951 effort=0.20 velocity=8.0677777442 -> lower=0 upper=2.0943951 effort=6.0 velocity=8.0677777442

File: URDF/mujoco/ability_hand_left.urdf (robot description, URDF)
Before this commit: robot ability_hand, 18 links, 17 joints
Joints:
- joint index_q1: limit lower=0 upper=2.0943951 effort=0.20 velocity=8.0677777442 -> lower=0 upper=2.0943951 effort=6.0 velocity=8.0677777442
- joint index_q2: limit lower=0.0 upper=2.6586 effort=0.20 velocity=8.0677777442 -> lower=0.0 upper=2.6586 effort=6.0 velocity=8.0677777442
- joint middle_q1: limit lower=0 upper=2.0943951 effort=0.20 velocity=8.0677777442 -> lower=0 upper=2.0943951 effort=6.0 velocity=8.0677777442
- joint middle_q2: limit lower=0.0 upper=2.6586 effort=0.20 velocity=8.0677777442 -> lower=0.0 upper=2.6586 effort=6.0 velocity=8.0677777442
- joint pinky_q1: limit lower=0 upper=2.0943951 effort=0.20 velocity=8.0677777442 -> lower=0 upper=2.0943951 effort=6.0 velocity=8.0677777442
- joint pinky_q2: limit lower=0.0 upper=2.6586 effort=0.20 velocity=8.0677777442 -> lower=0.0 upper=2.6586 effort=6.0 velocity=8.0677777442
- joint ring_q1: limit lower=0 upper=2.0943951 effort=0.20 velocity=8.0677777442 -> lower=0 upper=2.0943951 effort=6.0 velocity=8.0677777442
- joint ring_q2: limit lower=0.0 upper=2.6586 effort=0.20 velocity=8.0677777442 -> lower=0.0 upper=2.6586 effort=6.0 velocity=8.0677777442
- joint thumb_q1: limit lower=-2.0943951 upper=0 effort=0.20 velocity=8.0677777442 -> lower=-2.0943951 upper=0 effort=1.2 velocity=40.338888721
- joint thumb_q2: limit lower=0 upper=2.0943951 effort=0.20 velocity=8.0677777442 -> lower=0 upper=2.0943951 effort=6.0 velocity=8.0677777442

File: URDF/mujoco/ability_hand_right.urdf (robot description, URDF)
Before this commit: robot ability_hand, 18 links, 17 joints
Joints:
- joint index_q1: limit lower=0 upper=2.0943951 effort=0.20 velocity=8.0677777442 -> lower=0 upper=2.0943951 effort=6.0 velocity=8.0677777442
- joint index_q2: limit lower=0.0 upper=2.6586 effort=0.20 velocity=8.0677777442 -> lower=0.0 upper=2.6586 effort=6.0 velocity=8.0677777442
- joint middle_q1: limit lower=0 upper=2.0943951 effort=0.20 velocity=8.0677777442 -> lower=0 upper=2.0943951 effort=6.0 velocity=8.0677777442
- joint middle_q2: limit lower=0.0 upper=2.6586 effort=0.20 velocity=8.0677777442 -> lower=0.0 upper=2.6586 effort=6.0 velocity=8.0677777442
- joint pinky_q1: limit lower=0 upper=2.0943951 effort=0.20 velocity=8.0677777442 -> lower=0 upper=2.0943951 effort=6.0 velocity=8.0677777442
- joint pinky_q2: limit lower=0.0 upper=2.6586 effort=0.20 velocity=8.0677777442 -> lower=0.0 upper=2.6586 effort=6.0 velocity=8.0677777442
- joint ring_q1: limit lower=0 upper=2.0943951 effort=0.20 velocity=8.0677777442 -> lower=0 upper=2.0943951 effort=6.0 velocity=8.0677777442
- joint ring_q2: limit lower=0.0 upper=2.6586 effort=0.20 velocity=8.0677777442 -> lower=0.0 upper=2.6586 effort=6.0 velocity=8.0677777442
- joint thumb_q1: limit lower=-2.0943951 upper=0 effort=0.20 velocity=8.0677777442 -> lower=-2.0943951 upper=0 effort=1.2 velocity=40.338888721
- joint thumb_q2: limit lower=0 upper=2.0943951 effort=0.20 velocity=8.0677777442 -> lower=0 upper=2.0943951 effort=6.0 velocity=8.0677777442

Commit message: split thumb f2 into 2 now to make all mesh transforms 0

File: URDF/ability_hand_left.urdf (robot description, URDF)
Before this commit: robot ability_hand, 17 links, 16 joints
Links:
- link thumb_L2: geometry visual mesh filename=models/thumb-F2-left.STL

File: URDF/ability_hand_right.urdf (robot description, URDF)
Before this commit: robot ability_hand, 17 links, 16 joints
Links:
- link thumb_L2: geometry visual mesh filename=models/thumb-F2-right.STL
