Commit message: Update ability_hand_right_large.urdf
mesh file directory for index_L2 was incorrect

File: URDF/ability_hand_right_large.urdf (robot description, URDF)
Before this commit: robot ability_hand, 17 links, 16 joints
Links:
- link index_L2: geometry visual mesh filename=models/idx-F2-Lg.STL

Commit message: remove redundant link

File: URDF/ability_hand_right_large.urdf (robot description, URDF)
Before this commit: robot ability_hand, 47 links, 46 joints
Links:
- removed link thumb_base
- link base: geometry collision mesh filename=models/palm_hull_mir.STL; visual mesh filename=models/FB_palm_ref_MIR.STL
Joints:
- removed joint wrist2thumb
- joint thumb_q1: origin xyz= 0.0 0.0 0.0  rpy= 3.141592653589793 -0.0 -0.18884434641020664  -> xyz=-24.0476665e-3 3.78124745e-3 32.32964923e-3 rpy=-0.01675973 -0.08689062 -2.95079797; parent thumb_base -> base
