Commit message: remove redundant links

File: URDF/ability_hand_left_small.urdf (robot description, URDF)
Before this commit: robot ability_hand, 47 links, 46 joints
Links:
- removed link thumb_base
- link base: geometry collision mesh filename=models/palm_hull.STL; visual mesh filename=models/FB_palm_ref.STL
- link thumb_L1: geometry collision mesh filename=models/thumb-F1-hull.STL; visual mesh filename=models/thumb-F1.STL
- link thumb_L2: geometry collision mesh filename=models/thumb-F2-hull.STL; visual mesh filename=models/thumb-F2-left.STL
Joints:
- removed joint wrist2thumb
- joint thumb_q1: origin xyz=0 0 0 rpy=0 0 3.330437 -> xyz=24.0476665e-3 3.78124745e-3 32.32964923e-3 rpy=-3.1250458 -0.08693131 -0.1883423; parent thumb_base -> base

File: URDF/ability_hand_right_small.urdf (robot description, URDF)
Before this commit: robot ability_hand, 47 links, 46 joints
Links:
- removed link thumb_base
- link base: geometry collision mesh filename=models/palm_hull_mir.STL; visual mesh filename=models/FB_palm_ref_MIR.STL
Joints:
- removed joint wrist2thumb
- joint thumb_q1: origin xyz= 0.0 0.0 0.0  rpy= 3.141592653589793 -0.0 -0.18884434641020664  -> xyz=-24.0476665e-3 3.78124745e-3 32.32964923e-3 rpy=-0.01675973 -0.08689062 -2.95079797; parent thumb_base -> base
