Commit message: fixed urdf

File: URDF/ability_hand_right_small.urdf (robot description, URDF)
Before this commit: robot ability_hand, 17 links, 16 joints
Links:
- added link fsr0
- added link fsr1
- added link fsr10
- added link fsr11
- added link fsr12
- added link fsr13
- added link fsr14
- added link fsr15
- added link fsr16
- added link fsr17
- added link fsr18
- added link fsr19
- added link fsr2
- added link fsr20
- added link fsr21
- added link fsr22
- added link fsr23
- added link fsr24
- added link fsr25
- added link fsr26
- added link fsr27
- added link fsr28
- added link fsr29
- added link fsr3
- added link fsr4
- added link fsr5
- added link fsr6
- added link fsr7
- added link fsr8
- added link fsr9
- link base: mass 0.200 -> 0.37511000
- link index_L1: mass 0.00635888 -> 0.00636000; geometry collision mesh filename=models/idx-F1-hull.STL; visual mesh filename=models/idx-F1.STL
- link index_L2: mass 0.00645 -> 0.00600000; geometry collision mesh filename=models/idx-F2-hull.STL; visual mesh filename=models/idx-F2.STL
- link middle_L1: mass 0.00635888 -> 0.00636000; geometry collision mesh filename=models/idx-F1-hull.STL; visual mesh filename=models/idx-F1.STL
- link middle_L2: mass 0.00645 -> 0.00600000; geometry collision mesh filename=models/idx-F2-hull.STL; visual mesh filename=models/idx-F2.STL
- link pinky_L1: mass 0.00635888 -> 0.00636000; geometry collision mesh filename=models/idx-F1-hull.STL; visual mesh filename=models/idx-F1.STL
- link pinky_L2: mass 0.00645 -> 0.00600000; geometry collision mesh filename=models/idx-F2-hull.STL; visual mesh filename=models/idx-F2.STL
- link ring_L1: mass 0.00635888 -> 0.00636000; geometry collision mesh filename=models/idx-F1-hull.STL; visual mesh filename=models/idx-F1.STL
- link ring_L2: mass 0.00645 -> 0.00600000; geometry collision mesh filename=models/idx-F2-hull.STL; visual mesh filename=models/idx-F2.STL
- link thumb_L1: mass 0.00268342 -> 0.00200000; geometry collision mesh filename=models/thumb-F1-MIR-hull.STL; visual mesh filename=models/thumb-F1-MIR.STL
- link thumb_L2: mass 0.0055 -> 0.06000000; geometry collision mesh filename=models/thumb-F2-hull.STL; visual mesh filename=models/thumb-F2-right.STL
- link thumb_base: mass 0.200 -> None; geometry collision mesh filename=models/palm_hull_mir.STL; visual mesh filename=models/FB_palm_ref_MIR.STL
Joints:
- added joint fsr0: type fixed, parent index_L2, child fsr0, origin xyz=0.02556 -0.01391 -0.00435 rpy=3.14 0 -0.1848
- added joint fsr1: type fixed, parent index_L2, child fsr1, origin xyz=0.02517 -0.01110 -0.00000 rpy=-1.5708 0.0 -0.2316
- added joint fsr10: type fixed, parent middle_L2, child fsr10, origin xyz=0.01310 -0.00943 0.00435 rpy=0.00000 0.00000 -0.57199
- added joint fsr11: type fixed, parent middle_L2, child fsr11, origin xyz=0.03142 -0.01438 0.00000 rpy=-2.66907 -1.57080 0.00000
- added joint fsr12: type fixed, parent ring_L2, child fsr12, origin xyz=0.02556 -0.01391 -0.00435 rpy=3.14 0 -0.1848
- added joint fsr13: type fixed, parent ring_L2, child fsr13, origin xyz=0.02517 -0.01110 -0.00000 rpy=-1.5708 0.0 -0.2316
- added joint fsr14: type fixed, parent ring_L2, child fsr14, origin xyz=0.02556 -0.01391 0.00435 rpy=0.0 0.0 -0.1848036056311012
- added joint fsr15: type fixed, parent ring_L2, child fsr15, origin xyz=0.01310 -0.00943 -0.00435 rpy=3.14159 0.00000 -0.57092
- added joint fsr16: type fixed, parent ring_L2, child fsr16, origin xyz=0.01310 -0.00943 0.00435 rpy=0.00000 0.00000 -0.57199
- added joint fsr17: type fixed, parent ring_L2, child fsr17, origin xyz=0.03142 -0.01438 0.00000 rpy=-2.66907 -1.57080 0.00000
- added joint fsr18: type fixed, parent pinky_L2, child fsr18, origin xyz=0.02556 -0.01391 -0.00435 rpy=3.14 0 -0.1848
- added joint fsr19: type fixed, parent pinky_L2, child fsr19, origin xyz=0.02517 -0.01110 -0.00000 rpy=-1.5708 0.0 -0.2316
- added joint fsr2: type fixed, parent index_L2, child fsr2, origin xyz=0.02556 -0.01391 0.00435 rpy=0.0 0.0 -0.1848036056311012
- added joint fsr20: type fixed, parent pinky_L2, child fsr20, origin xyz=0.02556 -0.01391 0.00435 rpy=0.0 0.0 -0.1848036056311012
- added joint fsr21: type fixed, parent pinky_L2, child fsr21, origin xyz=0.01310 -0.00943 -0.00435 rpy=3.14159 0.00000 -0.57092
- added joint fsr22: type fixed, parent pinky_L2, child fsr22, origin xyz=0.01310 -0.00943 0.00435 rpy=0.00000 0.00000 -0.57199
- added joint fsr23: type fixed, parent pinky_L2, child fsr23, origin xyz=0.03142 -0.01438 0.00000 rpy=-2.66907 -1.57080 0.00000
- added joint fsr24: type fixed, parent thumb_L2, child fsr24, origin xyz=0.04747 0.01988 -0.001239 rpy=-2.29074 0.00001 0.41769
- added joint fsr25: type fixed, parent thumb_L2, child fsr25, origin xyz=0.04721 0.02124 0.006439 rpy=-1.30899 0.00001 0.41769
- added joint fsr26: type fixed, parent thumb_L2, child fsr26, origin xyz=0.04896 0.01654 0.01241 rpy=-0.32726 0.00001 0.41769
- added joint fsr27: type fixed, parent thumb_L2, child fsr27, origin xyz=0.03739 0.01536 -0.001289 rpy=-2.29074 0.00001 0.41769
- added joint fsr28: type fixed, parent thumb_L2, child fsr28, origin xyz=0.03888 0.01200 0.01244 rpy=-0.32726 0.00001 0.41769
- added joint fsr29: type fixed, parent thumb_L2, child fsr29, origin xyz=0.05591 0.02160 0.00558
- added joint fsr3: type fixed, parent index_L2, child fsr3, origin xyz=0.01310 -0.00943 -0.00435 rpy=3.14159 0.00000 -0.57092
- added joint fsr4: type fixed, parent index_L2, child fsr4, origin xyz=0.01310 -0.00943 0.00435 rpy=0.00000 0.00000 -0.57199
- added joint fsr5: type fixed, parent index_L2, child fsr5, origin xyz=0.03142 -0.01438 0.00000 rpy=-2.66907 -1.57080 0.00000
- added joint fsr6: type fixed, parent middle_L2, child fsr6, origin xyz=0.02556 -0.01391 -0.00435 rpy=3.14 0 -0.1848
- added joint fsr7: type fixed, parent middle_L2, child fsr7, origin xyz=0.02517 -0.01110 -0.00000 rpy=-1.5708 0.0 -0.2316
- added joint fsr8: type fixed, parent middle_L2, child fsr8, origin xyz=0.02556 -0.01391 0.00435 rpy=0.0 0.0 -0.1848036056311012
- added joint fsr9: type fixed, parent middle_L2, child fsr9, origin xyz=0.01310 -0.00943 -0.00435 rpy=3.14159 0.00000 -0.57092
- joint index_q1: origin xyz= 9.49e-3 -13.04e-3 -62.95e-3  rpy= -1.1595426535897932 1.284473 -1.0510016535897932  -> xyz=-2.8e-2 -9e-3 9.6e-2 rpy= 1.672 -1.317 -1.790 ; parent thumb_base -> base
- joint middle_q1: origin xyz= -9.653191e-3 -15.310271e-3 -67.853949e-3  rpy= -1.2810616535897934 1.308458 -1.2453756535897933  -> xyz= -0.008 -0.012 0.099  rpy= 1.513 -1.322 -1.558 ; parent thumb_base -> base
- joint pinky_q1: origin xyz= -49.521293e-3 -11.004583e-3 -63.029065e-3  rpy= -1.3764826535897934 1.32222 -1.4832096535897932  -> xyz= 0.031 -0.007 0.091  rpy= 1.410 -1.315 -1.313 ; parent thumb_base -> base
- joint ring_q1: origin xyz= -29.95426e-3 -14.212492e-3 -67.286105e-3  rpy= -1.424994653589793 1.321452 -1.4657306535897934  -> xyz= 0.012 -0.010 0.097  rpy= 1.361 -1.315 -1.330 ; parent thumb_base -> base

Commit message: add thumb coll, remove redud. link

File: URDF/ability_hand_left_large.urdf (robot description, URDF)
Before this commit: robot ability_hand, 47 links, 46 joints
Links:
- removed link thumb_base
- link base: geometry collision mesh filename=models/palm_hull.STL; visual mesh filename=models/FB_palm_ref.STL
- link thumb_L1: geometry collision mesh filename=models/thumb-F1-hull.STL; visual mesh filename=models/thumb-F1.STL
- link thumb_L2: geometry collision mesh filename=models/thumb-F2-hull.STL; visual mesh filename=models/thumb-F2-left.STL
Joints:
- removed joint wrist2thumb
- joint thumb_q1: origin xyz=0 0 0 rpy=0 0 3.330437 -> xyz=24.0476665e-3 3.78124745e-3 32.32964923e-3 rpy=-3.1250458 -0.08693131 -0.1883423; parent thumb_base -> base

Commit message: Fixed max ranges

File: URDF/ability_hand_left_large.urdf (robot description, URDF)
Before this commit: robot ability_hand, 46 links, 45 joints
Joints:
- joint index_q1: limit lower=0 upper=2.0943951 effort=6.0 velocity=8.0677777442 -> lower=0 upper=1.74 effort=6.0 velocity=8.0677777442
- joint index_q2: limit lower=0.0 upper=2.6586 effort=6.0 velocity=8.0677777442 -> lower=0.766 upper=2.61 effort=6.0 velocity=8.0677777442
- joint middle_q1: limit lower=0 upper=2.0943951 effort=6.0 velocity=8.0677777442 -> lower=0 upper=1.74 effort=6.0 velocity=8.0677777442
- joint middle_q2: limit lower=0.0 upper=2.6586 effort=6.0 velocity=8.0677777442 -> lower=0.766 upper=2.61 effort=6.0 velocity=8.0677777442
- joint pinky_q1: limit lower=0 upper=2.0943951 effort=6.0 velocity=8.0677777442 -> lower=0 upper=1.74 effort=6.0 velocity=8.0677777442
- joint pinky_q2: limit lower=0.0 upper=2.6586 effort=6.0 velocity=8.0677777442 -> lower=0.766 upper=2.61 effort=6.0 velocity=8.0677777442
- joint ring_q1: limit lower=0 upper=2.0943951 effort=6.0 velocity=8.0677777442 -> lower=0 upper=1.74 effort=6.0 velocity=8.0677777442
- joint ring_q2: limit lower=0.0 upper=2.6586 effort=6.0 velocity=8.0677777442 -> lower=0.766 upper=2.61 effort=6.0 velocity=8.0677777442
- joint thumb_q1: limit lower=-2.0943951 upper=0 effort=1.2 velocity=40.338888721 -> lower=-1.74 upper=0 effort=1.2 velocity=40.338888721
- joint thumb_q2: limit lower=0 upper=2.0943951 effort=6.0 velocity=8.0677777442 -> lower=0 upper=1.74 effort=6.0 velocity=8.0677777442

File: URDF/ability_hand_left_small.urdf (robot description, URDF)
Before this commit: robot ability_hand, 46 links, 45 joints
Joints:
- joint index_q1: limit lower=0 upper=2.0943951 effort=6.0 velocity=8.0677777442 -> lower=0 upper=1.74 effort=6.0 velocity=8.0677777442
- joint index_q2: limit lower=0.0 upper=2.6586 effort=6.0 velocity=8.0677777442 -> lower=0.766 upper=2.61 effort=6.0 velocity=8.0677777442
- joint middle_q1: limit lower=0 upper=2.0943951 effort=6.0 velocity=8.0677777442 -> lower=0 upper=1.74 effort=6.0 velocity=8.0677777442
- joint middle_q2: limit lower=0.0 upper=2.6586 effort=6.0 velocity=8.0677777442 -> lower=0.766 upper=2.61 effort=6.0 velocity=8.0677777442
- joint pinky_q1: limit lower=0 upper=2.0943951 effort=6.0 velocity=8.0677777442 -> lower=0 upper=1.74 effort=6.0 velocity=8.0677777442
- joint pinky_q2: limit lower=0.0 upper=2.6586 effort=6.0 velocity=8.0677777442 -> lower=0.766 upper=2.61 effort=6.0 velocity=8.0677777442
- joint ring_q1: limit lower=0 upper=2.0943951 effort=6.0 velocity=8.0677777442 -> lower=0 upper=1.74 effort=6.0 velocity=8.0677777442
- joint ring_q2: limit lower=0.0 upper=2.6586 effort=6.0 velocity=8.0677777442 -> lower=0.766 upper=2.61 effort=6.0 velocity=8.0677777442
- joint thumb_q1: limit lower=-2.0943951 upper=0 effort=1.2 velocity=40.338888721 -> lower=-1.74 upper=0 effort=1.2 velocity=40.338888721
- joint thumb_q2: limit lower=0 upper=2.0943951 effort=6.0 velocity=8.0677777442 -> lower=0 upper=1.74 effort=6.0 velocity=8.0677777442

File: URDF/ability_hand_right_large_no_fsr.urdf (robot description, URDF)
Before this commit: robot ability_hand, 46 links, 45 joints
Links:
- removed link fsr0
- removed link fsr1
- removed link fsr10
- removed link fsr11
- removed link fsr12
- removed link fsr13
- removed link fsr14
- removed link fsr15
- removed link fsr16
- removed link fsr17
- removed link fsr18
- removed link fsr19
- removed link fsr2
- removed link fsr20
- removed link fsr21
- removed link fsr22
- removed link fsr23
- removed link fsr24
- removed link fsr25
- removed link fsr26
- removed link fsr27
- removed link fsr28
- removed link fsr29
- removed link fsr3
- removed link fsr4
- removed link fsr5
- removed link fsr6
- removed link fsr7
- removed link fsr8
- removed link fsr9
Joints:
- removed joint fsr0
- removed joint fsr1
- removed joint fsr10
- removed joint fsr11
- removed joint fsr12
- removed joint fsr13
- removed joint fsr14
- removed joint fsr15
- removed joint fsr16
- removed joint fsr17
- removed joint fsr18
- removed joint fsr19
- removed joint fsr2
- removed joint fsr20
- removed joint fsr21
- removed joint fsr22
- removed joint fsr23
- removed joint fsr24
- removed joint fsr25
- removed joint fsr26
- removed joint fsr27
- removed joint fsr28
- removed joint fsr29
- removed joint fsr3
- removed joint fsr4
- removed joint fsr5
- removed joint fsr6
- removed joint fsr7
- removed joint fsr8
- removed joint fsr9

File: URDF/ability_hand_right_small.urdf (robot description, URDF)
Before this commit: robot ability_hand, 46 links, 45 joints
Joints:
- joint index_q1: limit lower=0 upper=2.0943951 effort=6.0 velocity=8.0677777442 -> lower=0 upper=1.74 effort=6.0 velocity=8.0677777442
- joint index_q2: limit lower=0.0 upper=2.6586 effort=6.0 velocity=8.0677777442 -> lower=0.766 upper=2.61 effort=6.0 velocity=8.0677777442
- joint middle_q1: limit lower=0 upper=2.0943951 effort=6.0 velocity=8.0677777442 -> lower=0 upper=1.74 effort=6.0 velocity=8.0677777442
- joint middle_q2: limit lower=0.0 upper=2.6586 effort=6.0 velocity=8.0677777442 -> lower=0.766 upper=2.61 effort=6.0 velocity=8.0677777442
- joint pinky_q1: limit lower=0 upper=2.0943951 effort=6.0 velocity=8.0677777442 -> lower=0 upper=1.74 effort=6.0 velocity=8.0677777442
- joint pinky_q2: limit lower=0.0 upper=2.6586 effort=6.0 velocity=8.0677777442 -> lower=0.766 upper=2.61 effort=6.0 velocity=8.0677777442
- joint ring_q1: limit lower=0 upper=2.0943951 effort=6.0 velocity=8.0677777442 -> lower=0 upper=1.74 effort=6.0 velocity=8.0677777442
- joint ring_q2: limit lower=0.0 upper=2.6586 effort=6.0 velocity=8.0677777442 -> lower=0.766 upper=2.61 effort=6.0 velocity=8.0677777442
- joint thumb_q1: limit lower=-2.0943951 upper=0 effort=1.2 velocity=40.338888721 -> lower=-1.74 upper=0 effort=1.2 velocity=40.338888721
- joint thumb_q2: limit lower=0 upper=2.0943951 effort=6.0 velocity=8.0677777442 -> lower=0 upper=1.74 effort=6.0 velocity=8.0677777442
