Commit message: better mimic offsets

File: URDF/ability_hand_left_large.urdf (robot description, URDF)
Before this commit: robot ability_hand, 46 links, 45 joints
Joints:
- joint fsr29: origin xyz=0.05591 0.02160 -0.00192 -> xyz=0.05591 0.02160 -0.00192 rpy=-1.39339 0.19354 -0.40280
- joint index_q1: limit lower=0 upper=1.74 effort=6.0 velocity=8.0677777442 -> lower=0.00 upper=1.74 effort=6.0 velocity=8.0677777442
- joint index_q2: limit lower=0.766 upper=2.61 effort=6.0 velocity=8.0677777442 -> lower=0.00 upper=1.844 effort=6.0 velocity=8.0677777442; mimic joint=index_q1 multiplier=1.05851325 offset=0.72349796 -> joint=index_q1 multiplier=1.05851325; origin xyz=38.472723e-3 3.257695e-3 0.000000e-3 rpy=0 0 0.084474 -> xyz=38.472723e-3 3.257695e-3 0.000000e-3 rpy=0 0 0.766
- joint middle_q1: limit lower=0 upper=1.74 effort=6.0 velocity=8.0677777442 -> lower=0.00 upper=1.74 effort=6.0 velocity=8.0677777442
- joint middle_q2: limit lower=0.766 upper=2.61 effort=6.0 velocity=8.0677777442 -> lower=0.00 upper=1.844 effort=6.0 velocity=8.0677777442; mimic joint=middle_q1 multiplier=1.05851325 offset=0.72349796 -> joint=middle_q1 multiplier=1.05851325; origin xyz=38.472723e-3 3.257695e-3 0.000000 rpy=0 0 0.084474 -> xyz=38.472723e-3 3.257695e-3 0.000000 rpy=0 0 0.766
- joint pinky_q1: limit lower=0 upper=1.74 effort=6.0 velocity=8.0677777442 -> lower=0.00 upper=1.74 effort=6.0 velocity=8.0677777442
- joint pinky_q2: limit lower=0.766 upper=2.61 effort=6.0 velocity=8.0677777442 -> lower=0.00 upper=1.844 effort=6.0 velocity=8.0677777442; mimic joint=pinky_q1 multiplier=1.05851325 offset=0.72349796 -> joint=pinky_q1 multiplier=1.05851325; origin xyz=38.472723e-3 3.257695e-3 0.000000 rpy=0 0 0.084474 -> xyz=38.472723e-3 3.257695e-3 0.000000 rpy=0 0 0.766
- joint ring_q1: limit lower=0 upper=1.74 effort=6.0 velocity=8.0677777442 -> lower=0.00 upper=1.74 effort=6.0 velocity=8.0677777442
- joint ring_q2: limit lower=0.766 upper=2.61 effort=6.0 velocity=8.0677777442 -> lower=0.00 upper=1.844 effort=6.0 velocity=8.0677777442; mimic joint=ring_q1 multiplier=1.05851325 offset=0.72349796 -> joint=ring_q1 multiplier=1.05851325; origin xyz=38.472723e-3 3.257695e-3 0.000000 rpy=0 0 0.084474 -> xyz=38.472723e-3 3.257695e-3 0.000000 rpy=0 0 0.766
- joint thumb_q2: limit lower=0 upper=1.74 effort=6.0 velocity=8.0677777442 -> lower=0.00 upper=1.74 effort=6.0 velocity=8.0677777442

File: URDF/ability_hand_left_small.urdf (robot description, URDF)
Before this commit: robot ability_hand, 46 links, 45 joints
Joints:
- joint index_q1: limit lower=0 upper=1.74 effort=6.0 velocity=8.0677777442 -> lower=0.00 upper=1.74 effort=6.0 velocity=8.0677777442
- joint index_q2: limit lower=0.766 upper=2.61 effort=6.0 velocity=8.0677777442 -> lower=0.00 upper=1.844 effort=6.0 velocity=8.0677777442; mimic joint=index_q1 multiplier=1.05851325 offset=0.72349796 -> joint=index_q1 multiplier=1.05851325; origin xyz=38.472723e-3 3.257695e-3 0.000000e-3 rpy=0 0 0.084474 -> xyz=38.472723e-3 3.257695e-3 0.000000e-3 rpy=0 0 0.766
- joint middle_q1: limit lower=0 upper=1.74 effort=6.0 velocity=8.0677777442 -> lower=0.00 upper=1.74 effort=6.0 velocity=8.0677777442
- joint middle_q2: limit lower=0.766 upper=2.61 effort=6.0 velocity=8.0677777442 -> lower=0.00 upper=1.844 effort=6.0 velocity=8.0677777442; mimic joint=middle_q1 multiplier=1.05851325 offset=0.72349796 -> joint=middle_q1 multiplier=1.05851325; origin xyz=38.472723e-3 3.257695e-3 0.000000 rpy=0 0 0.084474 -> xyz=38.472723e-3 3.257695e-3 0.000000 rpy=0 0 0.766
- joint pinky_q1: limit lower=0 upper=1.74 effort=6.0 velocity=8.0677777442 -> lower=0.00 upper=1.74 effort=6.0 velocity=8.0677777442
- joint pinky_q2: limit lower=0.766 upper=2.61 effort=6.0 velocity=8.0677777442 -> lower=0.00 upper=1.844 effort=6.0 velocity=8.0677777442; mimic joint=pinky_q1 multiplier=1.05851325 offset=0.72349796 -> joint=pinky_q1 multiplier=1.05851325; origin xyz=38.472723e-3 3.257695e-3 0.000000 rpy=0 0 0.084474 -> xyz=38.472723e-3 3.257695e-3 0.000000 rpy=0 0 0.766
- joint ring_q1: limit lower=0 upper=1.74 effort=6.0 velocity=8.0677777442 -> lower=0.00 upper=1.74 effort=6.0 velocity=8.0677777442
- joint ring_q2: limit lower=0.766 upper=2.61 effort=6.0 velocity=8.0677777442 -> lower=0.00 upper=1.844 effort=6.0 velocity=8.0677777442; mimic joint=ring_q1 multiplier=1.05851325 offset=0.72349796 -> joint=ring_q1 multiplier=1.05851325; origin xyz=38.472723e-3 3.257695e-3 0.000000 rpy=0 0 0.084474 -> xyz=38.472723e-3 3.257695e-3 0.000000 rpy=0 0 0.766
- joint thumb_q2: limit lower=0 upper=1.74 effort=6.0 velocity=8.0677777442 -> lower=0.00 upper=1.74 effort=6.0 velocity=8.0677777442

File: URDF/ability_hand_right_large.urdf (robot description, URDF)
Before this commit: robot ability_hand, 46 links, 45 joints
Joints:
- joint index_q1: limit lower=0 upper=1.74 effort=6.0 velocity=8.0677777442 -> lower=0.00 upper=1.74 effort=6.0 velocity=8.0677777442
- joint index_q2: limit lower=0.766 upper=2.61 effort=6.0 velocity=8.0677777442 -> lower=0.00 upper=1.844 effort=6.0 velocity=8.0677777442; mimic joint=index_q1 multiplier=1.05851325 offset=0.72349796 -> joint=index_q1 multiplier=1.05851325; origin xyz=38.472723e-3 3.257695e-3 0.000000e-3 rpy=0 0 0.084474 -> xyz=38.472723e-3 3.257695e-3 0.000000e-3 rpy=0 0 0.766
- joint middle_q1: limit lower=0 upper=1.74 effort=6.0 velocity=8.0677777442 -> lower=0.00 upper=1.74 effort=6.0 velocity=8.0677777442
- joint middle_q2: limit lower=0.766 upper=2.61 effort=6.0 velocity=8.0677777442 -> lower=0.00 upper=1.844 effort=6.0 velocity=8.0677777442; mimic joint=middle_q1 multiplier=1.05851325 offset=0.72349796 -> joint=middle_q1 multiplier=1.05851325; origin xyz=38.472723e-3 3.257695e-3 0.000000 rpy=0 0 0.084474 -> xyz=38.472723e-3 3.257695e-3 0.000000 rpy=0 0 0.766
- joint pinky_q1: limit lower=0 upper=1.74 effort=6.0 velocity=8.0677777442 -> lower=0.00 upper=1.74 effort=6.0 velocity=8.0677777442
- joint pinky_q2: limit lower=0.766 upper=2.61 effort=6.0 velocity=8.0677777442 -> lower=0.00 upper=1.844 effort=6.0 velocity=8.0677777442; mimic joint=pinky_q1 multiplier=1.05851325 offset=0.72349796 -> joint=pinky_q1 multiplier=1.05851325; origin xyz=38.472723e-3 3.257695e-3 0.000000 rpy=0 0 0.084474 -> xyz=38.472723e-3 3.257695e-3 0.000000 rpy=0 0 0.766
- joint ring_q1: limit lower=0 upper=1.74 effort=6.0 velocity=8.0677777442 -> lower=0.00 upper=1.74 effort=6.0 velocity=8.0677777442
- joint ring_q2: limit lower=0.766 upper=2.61 effort=6.0 velocity=8.0677777442 -> lower=0.00 upper=1.844 effort=6.0 velocity=8.0677777442; mimic joint=ring_q1 multiplier=1.05851325 offset=0.72349796 -> joint=ring_q1 multiplier=1.05851325; origin xyz=38.472723e-3 3.257695e-3 0.000000 rpy=0 0 0.084474 -> xyz=38.472723e-3 3.257695e-3 0.000000 rpy=0 0 0.766
- joint thumb_q2: limit lower=0 upper=1.74 effort=6.0 velocity=8.0677777442 -> lower=0.00 upper=1.74 effort=6.0 velocity=8.0677777442

File: URDF/ability_hand_right_large_no_fsr.urdf (robot description, URDF)
Before this commit: robot ability_hand, 16 links, 15 joints
Joints:
- joint index_q1: limit lower=0 upper=1.74 effort=6.0 velocity=8.0677777442 -> lower=0.00 upper=1.74 effort=6.0 velocity=8.0677777442
- joint index_q2: limit lower=0.766 upper=2.61 effort=6.0 velocity=8.0677777442 -> lower=0.00 upper=1.844 effort=6.0 velocity=8.0677777442; mimic joint=index_q1 multiplier=1.05851325 offset=0.72349796 -> joint=index_q1 multiplier=1.05851325; origin xyz=38.472723e-3 3.257695e-3 0.000000e-3 rpy=0 0 0.084474 -> xyz=38.472723e-3 3.257695e-3 0.000000e-3 rpy=0 0 0.766
- joint middle_q1: limit lower=0 upper=1.74 effort=6.0 velocity=8.0677777442 -> lower=0.00 upper=1.74 effort=6.0 velocity=8.0677777442
- joint middle_q2: limit lower=0.766 upper=2.61 effort=6.0 velocity=8.0677777442 -> lower=0.00 upper=1.844 effort=6.0 velocity=8.0677777442; mimic joint=middle_q1 multiplier=1.05851325 offset=0.72349796 -> joint=middle_q1 multiplier=1.05851325; origin xyz=38.472723e-3 3.257695e-3 0.000000 rpy=0 0 0.084474 -> xyz=38.472723e-3 3.257695e-3 0.000000 rpy=0 0 0.766
- joint pinky_q1: limit lower=0 upper=1.74 effort=6.0 velocity=8.0677777442 -> lower=0.00 upper=1.74 effort=6.0 velocity=8.0677777442
- joint pinky_q2: limit lower=0.766 upper=2.61 effort=6.0 velocity=8.0677777442 -> lower=0.00 upper=1.844 effort=6.0 velocity=8.0677777442; mimic joint=pinky_q1 multiplier=1.05851325 offset=0.72349796 -> joint=pinky_q1 multiplier=1.05851325; origin xyz=38.472723e-3 3.257695e-3 0.000000 rpy=0 0 0.084474 -> xyz=38.472723e-3 3.257695e-3 0.000000 rpy=0 0 0.766
- joint ring_q1: limit lower=0 upper=1.74 effort=6.0 velocity=8.0677777442 -> lower=0.00 upper=1.74 effort=6.0 velocity=8.0677777442
- joint ring_q2: limit lower=0.766 upper=2.61 effort=6.0 velocity=8.0677777442 -> lower=0.00 upper=1.844 effort=6.0 velocity=8.0677777442; mimic joint=ring_q1 multiplier=1.05851325 offset=0.72349796 -> joint=ring_q1 multiplier=1.05851325; origin xyz=38.472723e-3 3.257695e-3 0.000000 rpy=0 0 0.084474 -> xyz=38.472723e-3 3.257695e-3 0.000000 rpy=0 0 0.766
- joint thumb_q2: limit lower=0 upper=1.74 effort=6.0 velocity=8.0677777442 -> lower=0.00 upper=1.74 effort=6.0 velocity=8.0677777442

File: URDF/ability_hand_right_small.urdf (robot description, URDF)
Before this commit: robot ability_hand, 46 links, 45 joints
Joints:
- joint index_q1: limit lower=0 upper=1.74 effort=6.0 velocity=8.0677777442 -> lower=0.00 upper=1.74 effort=6.0 velocity=8.0677777442
- joint index_q2: limit lower=0.766 upper=2.61 effort=6.0 velocity=8.0677777442 -> lower=0.00 upper=1.844 effort=6.0 velocity=8.0677777442; mimic joint=index_q1 multiplier=1.05851325 offset=0.72349796 -> joint=index_q1 multiplier=1.05851325; origin xyz=38.472723e-3 3.257695e-3 0.000000e-3 rpy=0 0 0.084474 -> xyz=38.472723e-3 3.257695e-3 0.000000e-3 rpy=0 0 0.766
- joint middle_q1: limit lower=0 upper=1.74 effort=6.0 velocity=8.0677777442 -> lower=0.00 upper=1.74 effort=6.0 velocity=8.0677777442
- joint middle_q2: limit lower=0.766 upper=2.61 effort=6.0 velocity=8.0677777442 -> lower=0.00 upper=1.844 effort=6.0 velocity=8.0677777442; mimic joint=middle_q1 multiplier=1.05851325 offset=0.72349796 -> joint=middle_q1 multiplier=1.05851325; origin xyz=38.472723e-3 3.257695e-3 0.000000 rpy=0 0 0.084474 -> xyz=38.472723e-3 3.257695e-3 0.000000 rpy=0 0 0.766
- joint pinky_q1: limit lower=0 upper=1.74 effort=6.0 velocity=8.0677777442 -> lower=0.00 upper=1.74 effort=6.0 velocity=8.0677777442
- joint pinky_q2: limit lower=0.766 upper=2.61 effort=6.0 velocity=8.0677777442 -> lower=0.00 upper=1.844 effort=6.0 velocity=8.0677777442; mimic joint=pinky_q1 multiplier=1.05851325 offset=0.72349796 -> joint=pinky_q1 multiplier=1.05851325; origin xyz=38.472723e-3 3.257695e-3 0.000000 rpy=0 0 0.084474 -> xyz=38.472723e-3 3.257695e-3 0.000000 rpy=0 0 0.766
- joint ring_q1: limit lower=0 upper=1.74 effort=6.0 velocity=8.0677777442 -> lower=0.00 upper=1.74 effort=6.0 velocity=8.0677777442
- joint ring_q2: limit lower=0.766 upper=2.61 effort=6.0 velocity=8.0677777442 -> lower=0.00 upper=1.844 effort=6.0 velocity=8.0677777442; mimic joint=ring_q1 multiplier=1.05851325 offset=0.72349796 -> joint=ring_q1 multiplier=1.05851325; origin xyz=38.472723e-3 3.257695e-3 0.000000 rpy=0 0 0.084474 -> xyz=38.472723e-3 3.257695e-3 0.000000 rpy=0 0 0.766
- joint thumb_q2: limit lower=0 upper=1.74 effort=6.0 velocity=8.0677777442 -> lower=0.00 upper=1.74 effort=6.0 velocity=8.0677777442
