Commit message: added right hand mujoco. mimic relationship not preserved in mujoco compilations

File: URDF/mujoco/ability_hand_right.urdf (robot description, URDF)
Before this commit: robot ability_hand, 12 links, 11 joints
Links:
- link pinky_L1: geometry visual mesh filename=models/idx-F1-hull.STL
- link pinky_L2: geometry collision mesh filename=models/idx-F2-hull.STL
- link ring_L1: geometry collision mesh filename=models/idx-F1-hull.STL
- link ring_L2: geometry collision mesh filename=models/idx-F2-hull.STL
- link thumb_L1: geometry collision mesh filename=models/thumb-F1-MIR-hull.STL
- link thumb_L2: geometry collision mesh filename=models/thumb-F2-hull.STL
