Commit message: visuals to urdf added back and a fun little xml that flops two abh models on top of each other

File: URDF/mujoco/ability_hand_left.urdf (robot description, URDF)
Before this commit: robot ability_hand, 12 links, 11 joints
Links:
- link base: geometry collision mesh filename=palm_hull.STL; visual mesh filename=FB_palm_ref.STL
- link index_L1: geometry collision mesh filename=idx-F1-hull.STL; visual mesh filename=idx-F1.STL
- link index_L2: geometry collision mesh filename=idx-F2-hull.STL; visual mesh filename=idx-F2.STL
- link middle_L1: geometry collision mesh filename=idx-F1-hull.STL; visual mesh filename=idx-F1.STL
- link middle_L2: geometry collision mesh filename=idx-F2-hull.STL; visual mesh filename=idx-F2.STL
- link pinky_L1: geometry collision mesh filename=idx-F1-hull.STL; visual mesh filename=idx-F1.STL
- link pinky_L2: geometry collision mesh filename=idx-F2-hull.STL; visual mesh filename=idx-F2.STL
- link ring_L1: geometry collision mesh filename=idx-F1-hull.STL; visual mesh filename=idx-F1.STL
- link ring_L2: geometry collision mesh filename=idx-F2-hull.STL; visual mesh filename=idx-F2.STL
- link thumb_L1: geometry collision mesh filename=thumb-F1-hull.STL; visual mesh filename=thumb-F1.STL
- link thumb_L2: geometry collision mesh filename=thumb-F2-hull.STL; visual mesh filename=thumb-F2.STL

File: URDF/mujoco/ability_hand_right.urdf (robot description, URDF)
Before this commit: robot ability_hand, 12 links, 11 joints
Links:
- link base: geometry collision mesh filename=models/palm_hull_mir.STL; visual mesh filename=models/FB_palm_ref_MIR.STL
- link index_L1: geometry collision mesh filename=models/idx-F1-hull.STL; visual mesh filename=models/idx-F1.STL
- link index_L2: geometry collision mesh filename=models/idx-F2-hull.STL; visual mesh filename=models/idx-F2.STL
- link middle_L1: geometry collision mesh filename=models/idx-F1-hull.STL; visual mesh filename=models/idx-F1.STL
- link middle_L2: geometry collision mesh filename=models/idx-F2-hull.STL; visual mesh filename=models/idx-F2.STL
- link pinky_L1: geometry visual mesh filename=models/idx-F1-hull.STL; visual mesh filename=models/idx-F1.STL
- link pinky_L2: geometry collision mesh filename=models/idx-F2-hull.STL; visual mesh filename=models/idx-F2.STL
- link ring_L1: geometry collision mesh filename=models/idx-F1-hull.STL; visual mesh filename=models/idx-F1.STL
- link ring_L2: geometry collision mesh filename=models/idx-F2-hull.STL; visual mesh filename=models/idx-F2.STL
- link thumb_L1: geometry collision mesh filename=models/thumb-F1-MIR-hull.STL; visual mesh filename=models/thumb-F1-MIR.STL
- link thumb_L2: geometry collision mesh filename=models/thumb-F2-hull.STL; visual mesh filename=models/thumb-F2.STL

Commit message: update to mujoco urdfs, need to recompile

File: URDF/mujoco/ability_hand_left.urdf (robot description, URDF)
Before this commit: robot ability_hand, 12 links, 11 joints
Links:
- added link thumb_base, mass 0.400; collision mesh filename=palm_hull.STL; visual mesh filename=FB_palm_ref.STL
- link base: mass 0.400 -> 0.200; geometry visual mesh filename=wristmesh.STL
Joints:
- added joint wrist2thumb: type fixed, parent base, child thumb_base, origin xyz=24.0476665e-3 3.78124745e-3 32.32964923e-3 rpy=3.14148426 0.08848813 3.14036612
- joint index_q1: parent base -> thumb_base
- joint middle_q1: parent base -> thumb_base
- joint pinky_q1: parent base -> thumb_base
- joint ring_q1: parent base -> thumb_base
- joint thumb_q1: parent base -> thumb_base

File: URDF/mujoco/ability_hand_right.urdf (robot description, URDF)
Before this commit: robot ability_hand, 12 links, 11 joints
Links:
- added link thumb_base, mass 0.400; collision mesh filename=models/palm_hull_mir.STL; visual mesh filename=models/FB_palm_ref_MIR.STL
- link base: mass 0.400 -> 0.200; geometry visual mesh filename=models/wristmesh.STL
Joints:
- added joint wrist2thumb: type fixed, parent base, child thumb_base, origin xyz=-24.0476665e-3 3.78124745e-3 32.32964923e-3 rpy=3.14148426 -0.08848813 -3.14036612
- joint index_q1: parent base -> thumb_base
- joint middle_q1: parent base -> thumb_base
- joint pinky_q1: parent base -> thumb_base
- joint ring_q1: parent base -> thumb_base
- joint thumb_q1: parent base -> thumb_base

Commit message: mujoco urdf anchors

File: URDF/mujoco/ability_hand_left.urdf (robot description, URDF)
Before this commit: robot ability_hand, 13 links, 12 joints
Links:
- added link index_anchor
- added link middle_anchor
- added link pinky_anchor
- added link ring_anchor
- added link thumb_anchor
Joints:
- added joint idx_anchor: type fixed, parent index_L2, child index_anchor, origin xyz=31.5541e-3  -10.44e-3 0.14e-3 rpy=0 0 0
- added joint mid_anchor: type fixed, parent middle_L2, child middle_anchor, origin xyz=31.5541e-3  -10.44e-3 0.14e-3 rpy=0 0 0
- added joint pnky_anchor: type fixed, parent pinky_L2, child pinky_anchor, origin xyz=31.5541e-3  -10.44e-3 0.14e-3 rpy=0 0 0
- added joint rng_anchor: type fixed, parent ring_L2, child ring_anchor, origin xyz=31.5541e-3  -10.44e-3 0.14e-3 rpy=0 0 0
- added joint thmb_anchor: type fixed, parent thumb_L2, child thumb_anchor, origin xyz=52.0012259e-3  28.0086971e-3 -.884835778e-3 rpy=0 0 0

File: URDF/mujoco/ability_hand_right.urdf (robot description, URDF)
Before this commit: robot ability_hand, 13 links, 12 joints
Links:
- added link index_anchor
- added link middle_anchor
- added link pinky_anchor
- added link ring_anchor
- added link thumb_anchor
Joints:
- added joint idx_anchor: type fixed, parent index_L2, child index_anchor, origin xyz=31.5541e-3  -10.44e-3 0.14e-3 rpy=0 0 0
- added joint mid_anchor: type fixed, parent middle_L2, child middle_anchor, origin xyz=31.5541e-3  -10.44e-3 0.14e-3 rpy=0 0 0
- added joint pnky_anchor: type fixed, parent pinky_L2, child pinky_anchor, origin xyz=31.5541e-3  -10.44e-3 0.14e-3 rpy=0 0 0
- added joint rng_anchor: type fixed, parent ring_L2, child ring_anchor, origin xyz=31.5541e-3  -10.44e-3 0.14e-3 rpy=0 0 0
- added joint thmb_anchor: type fixed, parent thumb_L2, child thumb_anchor, origin xyz=52.00122724e-3 28.00869333e-3 6.98483578e-3 rpy=0 0 0
